File: lm335_voltage_cond.sch (KiCad schematic (older format))
At the start: 11 parts, among them U1 LM324AN

Commit message: c
Parts:
- added C1: C, ~, symbol C
- added D2: LED, ~, symbol LED
- added K1: OUT, symbol CONN_3
- added P1: CONN_1, symbol CONN_1
- added R8, R?: 2.2k, ~, symbol R
- added Z1: 2.5V, ~, symbol ZENER
- R7: renamed from R?; value 15.8k -> 2.2k
- gave numbers to parts that had none: 1
Connections:
- net +5V: now also C1.1, K1.1 (P1), R8.2, R?.1
- net GND: now also C1.2, D2.2 (K), K1.2 (PM), Z1.1 (A)
- net at R2.1, R5.2, U1.1: now also P1.1
- net at U1.3 (+): now also R8.1, Z1.2 (K)
- net OUT: now reaches R1.2, U1.7
- net OUT: now also K1.3 (P3)
- new net: D2.1 (A), R?.2
Changed lines of the file:
@@
 Connection ~ 4500 3150
 $Comp
-L GND #PWR?
+L GND #PWR01
 U 1 1 52D0CFE5
 P 2100 3800
-F 0 "#PWR?" H 2100 3800 30  0001 C CNN
+F 0 "#PWR01" H 2100 3800 30  0001 C CNN
 F 1 "GND" H 2100 3730 30  0001 C CNN
 F 2 "" H 2100 3800 60  0000 C CNN
@@
 $EndComp
 $Comp
-L GND #PWR?
+L GND #PWR02
 U 1 1 52D0CFF2
 P 4500 3950
-F 0 "#PWR?" H 4500 3950 30  0001 C CNN
+F 0 "#PWR02" H 4500 3950 30  0001 C CNN
 F 1 "GND" H 4500 3880 30  0001 C CNN
 F 2 "" H 4500 3950 60  0000 C CNN
@@
 	2100 3650 2100 3800
 $Comp
-L LM335 U?
+L LM335 U2
 U 1 1 52D0D243
 P 6450 2900
-F 0 "U?" H 6600 3200 60  0000 C CNN
+F 0 "U2" H 6600 3200 60  0000 C CNN
 F 1 "LM335" H 5950 2950 60  0000 C CNN
 F 2 "" H 6450 2900 60  0000 C CNN
@@
 $EndComp
 $Comp
-L +5V #PWR?
+L +5V #PWR03
 U 1 1 52D0D252
 P 6450 1700
-F 0 "#PWR?" H 6450 1790 20  0001 C CNN
+F 0 "#PWR03" H 6450 1790 20  0001 C CNN
 F 1 "+5V" H 6450 1790 30  0000 C CNN
 F 2 "" H 6450 1700 60  0000 C CNN
@@
 $EndComp
 $Comp
-L R R?
+L R R7
 U 1 1 52D0D25F
 P 6450 2150
-F 0 "R?" V 6530 2150 40  0000 C CNN
-F 1 "15.8k" V 6457 2151 40  0000 C CNN
+F 0 "R7" V 6530 2150 40  0000 C CNN
+F 1 "2.2k" V 6457 2151 40  0000 C CNN
 F 2 "~" V 6380 2150 30  0000 C CNN
 F 3 "~" H 6450 2150 30  0000 C CNN
@@
 	6450 2400 6450 2600
 $Comp
-L GND #PWR?
+L GND #PWR04
 U 1 1 52D0D2DA
 P 6450 3400
-F 0 "#PWR?" H 6450 3400 30  0001 C CNN
+F 0 "#PWR04" H 6450 3400 30  0001 C CNN
 F 1 "GND" H 6450 3330 30  0001 C CNN
 F 2 "" H 6450 3400 60  0000 C CNN
@@
 Connection ~ 6450 3300
 $Comp
-L +5V #PWR?
+L +5V #PWR05
 U 1 1 52D0D3A6
 P 2900 1900
-F 0 "#PWR?" H 2900 1990 20  0001 C CNN
+F 0 "#PWR05" H 2900 1990 20  0001 C CNN
 F 1 "+5V" H 2900 1990 30  0000 C CNN
 F 2 "" H 2900 1900 60  0000 C CNN
@@
 $EndComp
 $Comp
-L GND #PWR?
+L GND #PWR06
 U 1 1 52D0D3AC
 P 2900 2900
-F 0 "#PWR?" H 2900 2900 30  0001 C CNN
+F 0 "#PWR06" H 2900 2900 30  0001 C CNN
 F 1 "GND" H 2900 2830 30  0001 C CNN
 F 2 "" H 2900 2900 60  0000 C CNN
@@
 Wire Wire Line
 	2500 3050 2750 3050
+$Comp
+L CONN_3 K1
+U 1 1 52D0D4AF
+P 6450 4000
+F 0 "K1" V 6400 4000 50  0000 C CNN
+F 1 "OUT" V 6500 4000 40  0000 C CNN
+F 2 "" H 6450 4000 60  0000 C CNN
+F 3 "" H 6450 4000 60  0000 C CNN
+	1    6450 4000
+	1    0    0    -1
+$EndComp
+$Comp
+L +5V #PWR07
+U 1 1 52D0D4C8
+P 5900 3800
+F 0 "#PWR07" H 5900 3890 20  0001 C CNN
+F 1 "+5V" H 5900 3890 30  0000 C CNN
+F 2 "" H 5900 3800 60  0000 C CNN
+F 3 "" H 5900 3800 60  0000 C CNN
+	1    5900 3800
+	1    0    0    -1
+$EndComp
+Wire Wire Line
+	6100 3900 5900 3900
+Wire Wire Line
+	5900 3900 5900 3800
+$Comp
+L GND #PWR08
+U 1 1 52D0D4F5
+P 5650 4050
+F 0 "#PWR08" H 5650 4050 30  0001 C CNN
+F 1 "GND" H 5650 3980 30  0001 C CNN
+F 2 "" H 5650 4050 60  0000 C CNN
+F 3 "" H 5650 4050 60  0000 C CNN
+	1    5650 4050
+	1    0    0    -1
+$EndComp
+Wire Wire Line
+	5650 4050 5650 4000
+Wire Wire Line
+	5650 4000 6100 4000
+Text Label 5700 2300 0    60   ~ 0
+OUT
+Wire Wire Line
+	5600 2300 5700 2300
+Text Label 5850 4100 0    60   ~ 0
+OUT
+Wire Wire Line
+	5850 4100 6100 4100
+$Comp
+L CONN_1 P1
+U 1 1 52D0D57F
+P 4050 2100
+F 0 "P1" H 4130 2100 40  0000 L CNN
+F 1 "CONN_1" H 4050 2155 30  0001 C CNN
+F 2 "" H 4050 2100 60  0000 C CNN
+F 3 "" H 4050 2100 60  0000 C CNN
+	1    4050 2100
+	1    0    0    -1
+$EndComp
+Wire Wire Line
+	3900 2400 3900 2100
+$Comp
+L R R?
+U 1 1 52D0D68A
+P 8400 2150
+F 0 "R?" V 8480 2150 40  0000 C CNN
+F 1 "2.2k" V 8407 2151 40  0000 C CNN
+F 2 "~" V 8330 2150 30  0000 C CNN
+F 3 "~" H 8400 2150 30  0000 C CNN
+	1    8400 2150
+	1    0    0    -1
+$EndComp
+$Comp
+L +5V #PWR09
+U 1 1 52D0D690
+P 8400 1750
+F 0 "#PWR09" H 8400 1840 20  0001 C CNN
+F 1 "+5V" H 8400 1840 30  0000 C CNN
+F 2 "" H 8400 1750 60  0000 C CNN
+F 3 "" H 8400 1750 60  0000 C CNN
+	1    8400 1750
+	1    0    0    -1
+$EndComp
+$Comp
+L LED D2
+U 1 1 52D0D698
+P 8400 2750
+F 0 "D2" H 8400 2850 50  0000 C CNN
+F 1 "LED" H 8400 2650 50  0000 C CNN
+F 2 "~" H 8400 2750 60  0000 C CNN
+F 3 "~" H 8400 2750 60  0000 C CNN
+	1    8400 2750
+	0    1    1    0
+$EndComp
+Wire Wire Line
+	8400 1750 8400 1900
+Wire Wire Line
+	8400 2400 8400 2550
+$Comp
+L GND #PWR010
+U 1 1 52D0D70C
+P 8400 3250
+F 0 "#PWR010" H 8400 3250 30  0001 C CNN
+F 1 "GND" H 8400 3180 30  0001 C CNN
+F 2 "" H 8400 3250 60  0000 C CNN
+F 3 "" H 8400 3250 60  0000 C CNN
+	1    8400 3250
+	1    0    0    -1
+$EndComp
+Wire Wire Line
+	8400 2950 8400 3250
+$Comp
+L C C1
+U 1 1 52D0D775
+P 8850 2500
+F 0 "C1" H 8850 2600 40  0000 L CNN
+F 1 "C" H 8856 2415 40  0000 L CNN
+F 2 "~" H 8888 2350 30  0000 C CNN
+F 3 "~" H 8850 2500 60  0000 C CNN
+	1    8850 2500
+	1    0    0    -1
+$EndComp
+Wire Wire Line
+	8400 1800 8850 1800
+Wire Wire Line
+	8850 1800 8850 2300
+Connection ~ 8400 1800
+Wire Wire Line
+	8400 3100 8850 3100
+Wire Wire Line
+	8850 3100 8850 2700
+Connection ~ 8400 3100
+$Comp
+L ZENER Z1
+U 1 1 52D0D968
+P 1500 2550
+F 0 "Z1" H 1500 2650 50  0000 C CNN
+F 1 "2.5V" H 1500 2450 40  0000 C CNN
+F 2 "~" H 1500 2550 60  0000 C CNN
+F 3 "~" H 1500 2550 60  0000 C CNN
+	1    1500 2550
+	0    -1   -1   0
+$EndComp
+$Comp
+L R R8
+U 1 1 52D0D975
+P 1500 2000
+F 0 "R8" V 1580 2000 40  0000 C CNN
+F 1 "2.2k" V 1507 2001 40  0000 C CNN
+F 2 "~" V 1430 2000 30  0000 C CNN
+F 3 "~" H 1500 2000 30  0000 C CNN
+	1    1500 2000
+	-1   0    0    1
+$EndComp
+$Comp
+L +5V #PWR?
+U 1 1 52D0D993
+P 1500 1550
+F 0 "#PWR?" H 1500 1640 20  0001 C CNN
+F 1 "+5V" H 1500 1640 30  0000 C CNN
+F 2 "" H 1500 1550 60  0000 C CNN
+F 3 "" H 1500 1550 60  0000 C CNN
+	1    1500 1550
+	1    0    0    -1
+$EndComp
+Wire Wire Line
+	1500 1550 1500 1750
+Wire Wire Line
+	1500 2250 1500 2350
+Wire Wire Line
+	2500 2300 1500 2300
+Connection ~ 1500 2300
+$Comp
+L GND #PWR?
+U 1 1 52D0DA51
+P 1500 3000
+F 0 "#PWR?" H 1500 3000 30  0001 C CNN
+F 1 "GND" H 1500 2930 30  0001 C CNN
+F 2 "" H 1500 3000 60  0000 C CNN
+F 3 "" H 1500 3000 60  0000 C CNN
+	1    1500 3000
+	1    0    0    -1
+$EndComp
+Wire Wire Line
+	1500 2750 1500 3000
 $EndSCHEMATC

Commit message: Added netlist
Parts:
- gave numbers to parts that had none: 1
Changed lines of the file:
@@
 	3900 2400 3900 2100
 $Comp
-L R R?
+L R R9
 U 1 1 52D0D68A
 P 8400 2150
-F 0 "R?" V 8480 2150 40  0000 C CNN
+F 0 "R9" V 8480 2150 40  0000 C CNN
 F 1 "2.2k" V 8407 2151 40  0000 C CNN
 F 2 "~" V 8330 2150 30  0000 C CNN
@@
 $EndComp
 $Comp
-L +5V #PWR?
+L +5V #PWR011
 U 1 1 52D0D993
 P 1500 1550
-F 0 "#PWR?" H 1500 1640 20  0001 C CNN
+F 0 "#PWR011" H 1500 1640 20  0001 C CNN
 F 1 "+5V" H 1500 1640 30  0000 C CNN
 F 2 "" H 1500 1550 60  0000 C CNN
@@
 Connection ~ 1500 2300
 $Comp
-L GND #PWR?
+L GND #PWR012
 U 1 1 52D0DA51
 P 1500 3000
-F 0 "#PWR?" H 1500 3000 30  0001 C CNN
+F 0 "#PWR012" H 1500 3000 30  0001 C CNN
 F 1 "GND" H 1500 2930 30  0001 C CNN
 F 2 "" H 1500 3000 60  0000 C CNN

Commit message: Did some routing
Parts:
- removed Z1: 2.5V, ~, symbol ZENER
- added Z1: ADR5041, ~, symbol ADR5041
- U1: value LM324AN -> AD8554ARUZ
Connections:
- net GND: now also Z1.2 (A)
- net at R8.1, U1.3 (+): now also Z1.1 (K)
Changed lines of the file:
@@
 P 3000 2400
 F 0 "U1" H 3050 2600 60  0000 C CNN
-F 1 "LM324AN" H 3150 2200 50  0000 C CNN
+F 1 "AD8554ARUZ" H 3150 2200 50  0000 C CNN
 F 2 "" H 3000 2400 60  0000 C CNN
 F 3 "" H 3000 2400 60  0000 C CNN
@@
 P 5100 2300
 F 0 "U1" H 5150 2500 60  0000 C CNN
-F 1 "LM324AN" H 5250 2100 50  0000 C CNN
+F 1 "AD8554ARUZ" H 5250 2100 50  0000 C CNN
 F 2 "" H 5100 2300 60  0000 C CNN
 F 3 "" H 5100 2300 60  0000 C CNN
@@
 P 3250 3150
 F 0 "U1" H 3300 3350 60  0000 C CNN
-F 1 "LM324AN" H 3400 2950 50  0000 C CNN
+F 1 "AD8554ARUZ" H 3400 2950 50  0000 C CNN
 F 2 "" H 3250 3150 60  0000 C CNN
 F 3 "" H 3250 3150 60  0000 C CNN
@@
 Connection ~ 8400 3100
 $Comp
-L ZENER Z1
-U 1 1 52D0D968
-P 1500 2550
-F 0 "Z1" H 1500 2650 50  0000 C CNN
-F 1 "2.5V" H 1500 2450 40  0000 C CNN
-F 2 "~" H 1500 2550 60  0000 C CNN
-F 3 "~" H 1500 2550 60  0000 C CNN
-	1    1500 2550
-	0    -1   -1   0
-$EndComp
-$Comp
 L R R8
 U 1 1 52D0D975
@@
 Wire Wire Line
 	1500 2750 1500 3000
+$Comp
+L ADR5041 Z1
+U 1 1 52D18185
+P 1500 2550
+F 0 "Z1" H 1500 2650 50  0000 C CNN
+F 1 "ADR5041" H 1500 2450 40  0000 C CNN
+F 2 "~" H 1500 2550 60  0000 C CNN
+F 3 "~" H 1500 2550 60  0000 C CNN
+	1    1500 2550
+	0    -1   -1   0
+$EndComp
 $EndSCHEMATC
